File: pcb_design/esp8266_y.brd (EAGLE design)
At the start: 160 x 100 mm, 25 parts

Commit message: add files
Parts:
- moved U$5 147.5 mm to (52.1, 19.1)
- moved U$11 143.2 mm to (57.1, 23.9)
- moved U$10 134.9 mm to (57.2, 14.1)
- moved D1 120.5 mm to (55.6, 64.4), turned to 180 degrees
- moved U$13 111.0 mm to (57.3, 42.0)
- moved 7448_IC 109.4 mm to (66.0, 29.4), turned to 270 degrees
- moved U$8 105.5 mm to (52.2, 47.0)
- moved U$18 104.4 mm to (6.86, 20.5), turned to 180 degrees
- moved U$12 103.5 mm to (57.2, 32.4)
- moved U$7 103.0 mm to (52.5, 37.3)
- moved U$6 100.7 mm to (51.4, 28.4)
- moved U$16 88.2 mm to (7.01, 28.1), turned to 180 degrees
- moved U$2 76.7 mm to (46.6, 69.3), turned to 270 degrees
- moved U$17 76.4 mm to (4.88, 55.2)
- moved J1 72.3 mm to (6.26, 11.7)
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Connections:
- net 3V: now also U$1.11
- net VCC: no longer U$1.11
Routing:
- net GND: track 0.00 -> 347.9 mm
- net D: track 0.00 -> 108.4 mm
- net N$16: track 0.00 -> 85.6 mm
- net 5V: track 0.00 -> 83.4 mm
- net N$15: track 0.00 -> 82.3 mm
- net N$12: track 0.00 -> 81.5 mm
- net N$13: track 0.00 -> 80.7 mm
- net A: track 0.00 -> 78.0 mm
- net VCC: track 0.00 -> 72.6 mm
- net N$14: track 0.00 -> 67.2 mm
- net C: track 0.00 -> 56.9 mm
- net B: track 0.00 -> 48.6 mm
- net RST_BUTTON: track 0.00 -> 47.7 mm
- net N$18: track 0.00 -> 45.8 mm
- net N$17: track 0.00 -> 37.4 mm
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Other:
- board size 160 x 100 mm -> 85 x 75 mm
