File: pcb_design/esp8266_y.sch (EAGLE design)
At the start: 25 parts

Commit message: add files
Connections:
- net VCC: no longer U$1.3V
Other:
- moved on the sheet: 7448_IC, 7805, D1, J1, S1, S2, S3, U$10, U$11, U$12, U$13, U$5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
